File: ai03-pad-duplicate/ai03-pad-duplicate.kicad_sch (KiCad schematic)
At the start: 14 parts

Commit message: Complete the schematic
Parts:
- added D1, D2, D3, D4: D_Small, Diode_SMD:D_SOD-123, symbol Device:D_Small
- added F1: 500mA, Fuse:Fuse_1206_3216Metric, symbol Device:Polyfuse_Small
- added MX1, MX2, MX3, MX4: MX-NoLED, MX_Alps_Hybrid:MX-1U-NoLED, symbol MX_Alps_Hybrid:MX-NoLED
- added USB1: Molex-0548190589, random keyboard parts:Molex-0548190589, symbol random-keyboard-parts:Molex-0548190589
- C1, C2, C3, C4, C5, C6, C7: renamed from C?; footprint (none) -> Capacitor_SMD:C_0805_2012Metric
- R1, R2, R4: renamed from R?; footprint (none) -> Resistor_SMD:R_0805_2012Metric
- R3: renamed from R?; value R_Small -> 10k; footprint (none) -> Resistor_SMD:R_0805_2012Metric
- SW1: renamed from SW?; footprint (none) -> random keyboard parts:SKQG-1155865
- Y1: renamed from Y?; footprint (none) -> Crystal:Crystal_SMD_3225-4Pin_3.2x2.5mm
- gave numbers to parts that had none: 1
Connections:
- net +5V: now also F1.2
- net D+: now also USB1.3 (D+)
- net D-: now also USB1.4 (D-)
- net GND: now also USB1.1 (GND)
- new net: D3.2 (A), MX3.2 (ROW)
- new net: D2.2 (A), MX2.2 (ROW)
- new net: D4.2 (A), MX4.2 (ROW)
- new net: D1.2 (A), MX1.2 (ROW)
- new net COL0: MX1.1 (COL), MX2.1 (COL)
- new net COL1: MX3.1 (COL), MX4.1 (COL)
- new net ROW0: D1.1 (K), D3.1 (K)
- new net ROW1: D2.1 (K), D4.1 (K)
- new net VCC: F1.1, USB1.5 (VBUS)

Commit message: Complete the PCB
Connections:
- net +5VP is gone; now on net +5V: R3.1
- net COL0: now also U1.40 (PF1)
- net COL1: now also U1.41 (PF0)
- net ROW0: now also U1.38 (PF5)
- net ROW1: now also U1.39 (PF4)
Changed lines of the file:
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@@
     (effects (font (size 1.27 1.27)) (justify right))
+  )
+  (global_label "COL1" (shape input) (at 88.9 111.76 0)
+    (effects (font (size 1.27 1.27)) (justify left))
+  )
+  (global_label "COL0" (shape input) (at 88.9 114.3 0)
+    (effects (font (size 1.27 1.27)) (justify left))
+  )
+  (global_label "ROW1" (shape input) (at 88.9 116.84 0)
+    (effects (font (size 1.27 1.27)) (justify left))
+  )
+  (global_label "ROW0" (shape input) (at 88.9 119.38 0)
+    (effects (font (size 1.27 1.27)) (justify left))
   )
   (global_label "D-" (shape input) (at 152.4 90.17 0)
@@
     )
   )
-  (symbol (lib_id "power:+5VP") (at 57.15 36.83 0) (unit 1)
+  (symbol (lib_id "power:+5V") (at 57.15 36.83 0) (unit 1)
     (property "Reference" "#PWR0108" (id 0) (at 57.15 40.64 0)
       (effects (font (size 1.27 1.27)) hide)
     )
-    (property "Value" "+5VP" (id 1) (at 57.5183 32.5056 0))
+    (property "Value" "+5V" (id 1) (at 57.5183 32.5056 0))
     (property "Footprint" "" (id 2) (at 57.15 36.83 0)
       (effects (font (size 1.27 1.27)) hide)
@@
       (reference "#PWR0107") (unit 1)
     )
-    (path "/cbd03ad9-7aa5-49c1-af9d-785a1226f2bb"
+    (path "/dfd25dd4-8d73-4896-8bad-98dd03fd9aca"
       (reference "#PWR0108") (unit 1)
     )

Commit message: Complete the PCB
Connections:
- net COL0: now also U1.9 (PB1); no longer U1.40 (PF1)
- net COL1: now also U1.8 (PB0); no longer U1.41 (PF0)
- net GND: now also C1.2, C2.2, USB1.6 (SHIELD); no longer C1.1, C2.1
- net ROW0: now also U1.10 (PB2); no longer U1.38 (PF5)
- net ROW1: now also U1.11 (PB3); no longer U1.39 (PF4)
- net at U1.17 (XTAL1), Y1.3: now also C1.1; no longer C1.2
- net at U1.16 (XTAL2), Y1.1: now also C2.1; no longer C2.2
Other:
- moved on the sheet: C1, C2
Changed lines of the file:
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@@
   (junction (at 139.7 54.61))
   (junction (at 139.7 59.69))
+  (junction (at 149.86 97.79))
   (junction (at 151.13 87.63))
   (junction (at 152.4 54.61))
@@
     (stroke (width 0) (type solid) (color 0 0 0 0))
   )
+  (wire (pts (xy 144.78 85.09) (xy 149.86 85.09))
+    (stroke (width 0) (type solid) (color 0 0 0 0))
+  )
   (wire (pts (xy 144.78 87.63) (xy 151.13 87.63))
     (stroke (width 0) (type solid) (color 0 0 0 0))
@@
     (stroke (width 0) (type solid) (color 0 0 0 0))
   )
-  (wire (pts (xy 144.78 97.79) (xy 154.94 97.79))
+  (wire (pts (xy 144.78 97.79) (xy 149.86 97.79))
+    (stroke (width 0) (type solid) (color 0 0 0 0))
+  )
+  (wire (pts (xy 149.86 85.09) (xy 149.86 97.79))
+    (stroke (width 0) (type solid) (color 0 0 0 0))
+  )
+  (wire (pts (xy 149.86 97.79) (xy 154.94 97.79))
     (stroke (width 0) (type solid) (color 0 0 0 0))
   )
@@
     (effects (font (size 1.27 1.27)) (justify right))
   )
-  (global_label "COL1" (shape input) (at 88.9 111.76 0)
-    (effects (font (size 1.27 1.27)) (justify left))
-  )
-  (global_label "COL0" (shape input) (at 88.9 114.3 0)
-    (effects (font (size 1.27 1.27)) (justify left))
-  )
-  (global_label "ROW1" (shape input) (at 88.9 116.84 0)
-    (effects (font (size 1.27 1.27)) (justify left))
-  )
-  (global_label "ROW0" (shape input) (at 88.9 119.38 0)
+  (global_label "COL1" (shape input) (at 88.9 50.8 0)
+    (effects (font (size 1.27 1.27)) (justify left))
+  )
+  (global_label "COL0" (shape input) (at 88.9 53.34 0)
+    (effects (font (size 1.27 1.27)) (justify left))
+  )
+  (global_label "ROW0" (shape input) (at 88.9 55.88 0)
+    (effects (font (size 1.27 1.27)) (justify left))
+  )
+  (global_label "ROW1" (shape input) (at 88.9 58.42 0)
     (effects (font (size 1.27 1.27)) (justify left))
   )
@@
     )
   )
-  (symbol (lib_id "Device:C_Small") (at 27.94 50.8 90) (unit 1)
-    (property "Reference" "C1" (id 0) (at 27.94 45.0277 90))
-    (property "Value" "22pF" (id 1) (at 27.94 47.3264 90))
+  (symbol (lib_id "Device:C_Small") (at 27.94 50.8 270) (unit 1)
+    (property "Reference" "C1" (id 0) (at 27.94 56.5723 90))
+    (property "Value" "22pF" (id 1) (at 27.94 54.2736 90))
     (property "Footprint" "Capacitor_SMD:C_0805_2012Metric" (id 2) (at 27.94 50.8 0)
       (effects (font (size 1.27 1.27)) hide)
@@
     )
   )
-  (symbol (lib_id "Device:C_Small") (at 27.94 59.69 90) (unit 1)
-    (property "Reference" "C2" (id 0) (at 27.94 53.9177 90))
-    (property "Value" "22pF" (id 1) (at 27.94 56.2164 90))
+  (symbol (lib_id "Device:C_Small") (at 27.94 59.69 270) (unit 1)
+    (property "Reference" "C2" (id 0) (at 27.94 65.4623 90))
+    (property "Value" "22pF" (id 1) (at 27.94 63.1636 90))
     (property "Footprint" "Capacitor_SMD:C_0805_2012Metric" (id 2) (at 27.94 59.69 0)
       (effects (font (size 1.27 1.27)) hide)
